File: 1LFO.sch (EAGLE design)
At the start: 26 parts, among them IC1 LM324D

Commit message: Use 3mm LED package (fits on board, panel still has 5mm hole).
Parts:
- LED1: device led:LED5MM -> led:LED3MM
Changed lines of the file:
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@@
 <part name="D2" library="diode" deviceset="DIODE-" device="DO214AA" value="DIODE"/>
 <part name="R7" library="rcl" deviceset="R-US_" device="R0603" value="10k"/>
-<part name="LED1" library="led" deviceset="LED" device="5MM"/>
+<part name="LED1" library="led" deviceset="LED" device="3MM"/>
 <part name="GND9" library="supply1" deviceset="GND" device=""/>
 </parts>

Commit message: Removed C7. Moved remaining timing caps a bit and changed value to the right one (10uF). Only one of C1 and C6 needs to be fitted. 10uF caps are easier to find in 1206 packages with higher voltage tolerances (should be >= 16V).
Parts:
- removed C7: 1u, rcl:C-USC0603K
- C1, C6: value 1u -> 10u
Connections:
- net N$1: no longer C7.1
- net TRI: no longer C7.2
Changed lines of the file:
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@@
 <part name="FRAME1" library="frames" deviceset="A4L-LOC" device=""/>
 <part name="IC1" library="linear" deviceset="LM324" device="D"/>
-<part name="C1" library="rcl" deviceset="C-US" device="C1206K" value="1u"/>
+<part name="C1" library="rcl" deviceset="C-US" device="C1206K" value="10u"/>
 <part name="C2" library="rcl" deviceset="C-US" device="C0603K" value="100n"/>
 <part name="C3" library="rcl" deviceset="C-US" device="C0603K" value="100n"/>
@@
 <part name="P+1" library="supply1" deviceset="+12V" device=""/>
 <part name="P-1" library="supply1" deviceset="-12V" device=""/>
-<part name="C6" library="rcl" deviceset="C-US" device="C0603K" value="1u"/>
-<part name="C7" library="rcl" deviceset="C-US" device="C0603K" value="1u"/>
+<part name="C6" library="rcl" deviceset="C-US" device="C0603K" value="10u"/>
 <part name="GND6" library="supply1" deviceset="GND" device=""/>
 <part name="R5" library="rcl" deviceset="R-US_" device="R0603" value="100k"/>
@@
 <instance part="P-1" gate="1" x="129.54" y="12.7"/>
 <instance part="C6" gate="G$1" x="43.18" y="106.68" rot="R90"/>
-<instance part="C7" gate="G$1" x="43.18" y="114.3" rot="R90"/>
 <instance part="GND6" gate="1" x="167.64" y="124.46" rot="R180"/>
 <instance part="R5" gate="G$1" x="160.02" y="114.3" rot="R180"/>
@@
 <pinref part="C6" gate="G$1" pin="1"/>
 <wire x1="35.56" y1="106.68" x2="40.64" y2="106.68" width="0.1524" layer="91"/>
-<wire x1="35.56" y1="106.68" x2="35.56" y2="114.3" width="0.1524" layer="91"/>
-<pinref part="C7" gate="G$1" pin="1"/>
-<wire x1="35.56" y1="114.3" x2="40.64" y2="114.3" width="0.1524" layer="91"/>
-<junction x="35.56" y="106.68"/>
 <junction x="35.56" y="99.06"/>
 </segment>
@@
 <wire x1="48.26" y1="106.68" x2="55.88" y2="106.68" width="0.1524" layer="91"/>
 <wire x1="55.88" y1="106.68" x2="55.88" y2="99.06" width="0.1524" layer="91"/>
-<wire x1="55.88" y1="106.68" x2="55.88" y2="114.3" width="0.1524" layer="91"/>
-<pinref part="C7" gate="G$1" pin="2"/>
-<wire x1="48.26" y1="114.3" x2="55.88" y2="114.3" width="0.1524" layer="91"/>
-<junction x="55.88" y="106.68"/>
 <junction x="55.88" y="99.06"/>
 <wire x1="55.88" y1="83.82" x2="55.88" y2="73.66" width="0.1524" layer="91"/>
